File: Jove.kicad_pcb (KiCad board)
At the start: 2 copper layers, 65 x 100 mm, 155 parts, among them J1 PJ301B, J2 PJ301B, J3 PJ301B, J4 PJ301B, J5 PJ301B, J6 PJ301B, P1 CONN_02X05, Q1 BCM857BS, Q2 BCM857BS, Q3 J112, Q4 J112, Q5 J112, Q6 J112, SW1 KS-01Q, U1 TL072-, U10 CD4027, U11 CD40106, U12 TS321, U13 TS321, U2 TL072-, U3 TL072-, U4 TL072-, U5 LM13700, U6 LM13700, U7 LM13700, U8 DG409, U9 CD4052

Commit message: panelized
Parts:
- added C1: 22pF, MyModules:SM0603-C-JRL, B.Cu at (236.0, 47.0)
- added C1: 22pF, MyModules:SM0603-C-JRL, B.Cu at (171.0, 47.0)
- added C1: 22pF, MyModules:SM0603-C-JRL, B.Cu at (106.0, 47.0)
- added C10: 10μF, Capacitors_SMD:c_elec_5x5.3, B.Cu at (254.0, 73.8)
- added C10: 10μF, Capacitors_SMD:c_elec_5x5.3, B.Cu at (189.0, 73.8)
- added C10: 10μF, Capacitors_SMD:c_elec_5x5.3, B.Cu at (124.0, 73.8)
- added C11: 22pF, MyModules:SM0603-C-JRL, B.Cu at (246.5, 84.0)
- added C11: 22pF, MyModules:SM0603-C-JRL, B.Cu at (181.5, 84.0)
- added C11: 22pF, MyModules:SM0603-C-JRL, B.Cu at (116.5, 84.0)
- added C12: 100n, MyModules:SM0603-C-JRL, B.Cu at (243.0, 44.8)
- added C12: 100n, MyModules:SM0603-C-JRL, B.Cu at (178.0, 44.8)
- added C12: 100n, MyModules:SM0603-C-JRL, B.Cu at (113.0, 44.8)
- added C13: 100n, MyModules:SM0603-C-JRL, B.Cu at (240.8, 39.0)
- added C13: 100n, MyModules:SM0603-C-JRL, B.Cu at (175.8, 39.0)
- added C13: 100n, MyModules:SM0603-C-JRL, B.Cu at (110.8, 39.0)
- added C14: 100n, MyModules:SM0603-C-JRL, B.Cu at (234.2, 31.8)
- added C14: 100n, MyModules:SM0603-C-JRL, B.Cu at (169.2, 31.8)
- added C14: 100n, MyModules:SM0603-C-JRL, B.Cu at (104.2, 31.8)
- added C15: 100n, MyModules:SM0603-C-JRL, B.Cu at (232.8, 17.0)
- added C15: 100n, MyModules:SM0603-C-JRL, B.Cu at (167.8, 17.0)
- added C15: 100n, MyModules:SM0603-C-JRL, B.Cu at (102.8, 17.0)
- added C16: 100n, MyModules:SM0603-C-JRL, B.Cu at (212.7, 50.2)
- added C16: 100n, MyModules:SM0603-C-JRL, B.Cu at (147.7, 50.2)
- added C16: 100n, MyModules:SM0603-C-JRL, B.Cu at (82.7, 50.2)
- added C17: 100n, MyModules:SM0603-C-JRL, B.Cu at (221.0, 56.0)
- added C17: 100n, MyModules:SM0603-C-JRL, B.Cu at (156.0, 56.0)
- added C17: 100n, MyModules:SM0603-C-JRL, B.Cu at (91.0, 56.0)
- added C18: 330pF, MyModules:CAP-BOX-PFR-5MM, B.Cu at (230.5, 91.5)
- added C18: 330pF, MyModules:CAP-BOX-PFR-5MM, B.Cu at (165.5, 91.5)
- added C18: 330pF, MyModules:CAP-BOX-PFR-5MM, B.Cu at (100.5, 91.5)
- added C19: 100n, MyModules:SM0603-C-JRL, B.Cu at (246.8, 87.5)
- added C19: 100n, MyModules:SM0603-C-JRL, B.Cu at (181.8, 87.5)
- added C19: 100n, MyModules:SM0603-C-JRL, B.Cu at (116.8, 87.5)
- added C2: 47pF, MyModules:SM0603-C-JRL, B.Cu at (221.0, 59.2)
- added C2: 47pF, MyModules:SM0603-C-JRL, B.Cu at (156.0, 59.2)
- added C2: 47pF, MyModules:SM0603-C-JRL, B.Cu at (91.0, 59.2)
- added C20: 100n, MyModules:SM0603-C-JRL, B.Cu at (232.5, 74.0)
- added C20: 100n, MyModules:SM0603-C-JRL, B.Cu at (167.5, 74.0)
- added C20: 100n, MyModules:SM0603-C-JRL, B.Cu at (102.5, 74.0)
- added C21: 0.47μ, MyModules:SM0603-C-JRL, B.Cu at (254.2, 32.5)
- added C21: 0.47μ, MyModules:SM0603-C-JRL, B.Cu at (189.2, 32.5)
- added C21: 0.47μ, MyModules:SM0603-C-JRL, B.Cu at (124.2, 32.5)
- added C22: 0.47μ, MyModules:SM0603-C-JRL, B.Cu at (262.2, 32.8)
- added C22: 0.47μ, MyModules:SM0603-C-JRL, B.Cu at (197.2, 32.8)
- added C22: 0.47μ, MyModules:SM0603-C-JRL, B.Cu at (132.2, 32.8)
- added C23: 10μF, Capacitors_SMD:c_elec_5x5.3, B.Cu at (267.2, 15.5)
- added C23: 10μF, Capacitors_SMD:c_elec_5x5.3, B.Cu at (202.2, 15.5)
- added C23: 10μF, Capacitors_SMD:c_elec_5x5.3, B.Cu at (137.2, 15.5)
- added C24: 10μF, Capacitors_SMD:c_elec_5x5.3, B.Cu at (267.2, 52.0)
- added C24: 10μF, Capacitors_SMD:c_elec_5x5.3, B.Cu at (202.2, 52.0)
- added C24: 10μF, Capacitors_SMD:c_elec_5x5.3, B.Cu at (137.2, 52.0)
- added C25: 330pF, MyModules:CAP-BOX-PFR-5MM, B.Cu at (248.5, 91.5)
- added C25: 330pF, MyModules:CAP-BOX-PFR-5MM, B.Cu at (183.5, 91.5)
- added C25: 330pF, MyModules:CAP-BOX-PFR-5MM, B.Cu at (118.5, 91.5)
- added C26: 100n, MyModules:SM0603-C-JRL, B.Cu at (217.5, 19.0)
- added C26: 100n, MyModules:SM0603-C-JRL, B.Cu at (152.5, 19.0)
- added C26: 100n, MyModules:SM0603-C-JRL, B.Cu at (87.5, 19.0)
- added C27: 100n, MyModules:SM0603-C-JRL, B.Cu at (224.0, 25.0)
- added C27: 100n, MyModules:SM0603-C-JRL, B.Cu at (159.0, 25.0)
- added C27: 100n, MyModules:SM0603-C-JRL, B.Cu at (94.0, 25.0)
- added C28: 22pF, MyModules:SM0603-C-JRL, B.Cu at (225.0, 50.9)
- added C28: 22pF, MyModules:SM0603-C-JRL, B.Cu at (160.0, 50.9)
- added C28: 22pF, MyModules:SM0603-C-JRL, B.Cu at (95.0, 50.9)
- added C29: 22pF, MyModules:SM0603-C-JRL, B.Cu at (223.7, 17.7)
- added C29: 22pF, MyModules:SM0603-C-JRL, B.Cu at (158.7, 17.7)
- added C29: 22pF, MyModules:SM0603-C-JRL, B.Cu at (93.7, 17.7)
- added C3: 4.7pF, MyModules:SM0603-C-JRL, B.Cu at (246.5, 41.0)
- added C3: 4.7pF, MyModules:SM0603-C-JRL, B.Cu at (181.5, 41.0)
- added C3: 4.7pF, MyModules:SM0603-C-JRL, B.Cu at (116.5, 41.0)
- added C4: 33pF, MyModules:SM0603-C-JRL, B.Cu at (243.0, 47.0)
- added C4: 33pF, MyModules:SM0603-C-JRL, B.Cu at (178.0, 47.0)
- added C4: 33pF, MyModules:SM0603-C-JRL, B.Cu at (113.0, 47.0)
- added C5: 47pF, MyModules:SM0603-C-JRL, B.Cu at (236.2, 21.0)
- added C5: 47pF, MyModules:SM0603-C-JRL, B.Cu at (171.2, 21.0)
- added C5: 47pF, MyModules:SM0603-C-JRL, B.Cu at (106.2, 21.0)
- added C6: 330pF, MyModules:CAP-BOX-PFR-5MM, B.Cu at (248.5, 61.5)
- added C6: 330pF, MyModules:CAP-BOX-PFR-5MM, B.Cu at (183.5, 61.5)
- added C6: 330pF, MyModules:CAP-BOX-PFR-5MM, B.Cu at (118.5, 61.5)
- added C7: 330pF, MyModules:CAP-BOX-PFR-5MM, B.Cu at (230.5, 61.5)
- added C7: 330pF, MyModules:CAP-BOX-PFR-5MM, B.Cu at (165.5, 61.5)
- added C7: 330pF, MyModules:CAP-BOX-PFR-5MM, B.Cu at (100.5, 61.5)
- added C8: 4.7pF, MyModules:SM0603-C-JRL, B.Cu at (228.0, 83.5)
- added C8: 4.7pF, MyModules:SM0603-C-JRL, B.Cu at (163.0, 83.5)
- added C8: 4.7pF, MyModules:SM0603-C-JRL, B.Cu at (98.0, 83.5)
- added C9: 33pF, MyModules:SM0603-C-JRL, B.Cu at (232.5, 79.5)
- added C9: 33pF, MyModules:SM0603-C-JRL, B.Cu at (167.5, 79.5)
- added C9: 33pF, MyModules:SM0603-C-JRL, B.Cu at (102.5, 79.5)
- added D1: LED, MyModules:3MM-LED-C1A2, F.Cu at (239.5, 13.0)
- added D1: LED, MyModules:3MM-LED-C1A2, F.Cu at (174.5, 13.0)
- added D1: LED, MyModules:3MM-LED-C1A2, F.Cu at (109.5, 13.0)
- added D10: 1N914, MyModules:SOD323-C1A2, B.Cu at (210.5, 53.2)
- added D10: 1N914, MyModules:SOD323-C1A2, B.Cu at (145.5, 53.2)
- added D10: 1N914, MyModules:SOD323-C1A2, B.Cu at (80.5, 53.2)
- added D2: LED, MyModules:3MM-LED-C1A2, F.Cu at (239.5, 18.0)
- added D2: LED, MyModules:3MM-LED-C1A2, F.Cu at (174.5, 18.0)
- added D2: LED, MyModules:3MM-LED-C1A2, F.Cu at (109.5, 18.0)
- added D3: LED, MyModules:3MM-LED-C1A2, F.Cu at (174.5, 23.0)
- added D3: LED, MyModules:3MM-LED-C1A2, F.Cu at (239.5, 23.0)
- added D3: LED, MyModules:3MM-LED-C1A2, F.Cu at (109.5, 23.0)
- added D4: LED, MyModules:3MM-LED-C1A2, F.Cu at (239.5, 28.0)
- added D4: LED, MyModules:3MM-LED-C1A2, F.Cu at (174.5, 28.0)
- added D4: LED, MyModules:3MM-LED-C1A2, F.Cu at (109.5, 28.0)
- added D5: 1N914, MyModules:SOD323-C1A2, B.Cu at (232.0, 81.5)
- added D5: 1N914, MyModules:SOD323-C1A2, B.Cu at (167.0, 81.5)
- added D5: 1N914, MyModules:SOD323-C1A2, B.Cu at (102.0, 81.5)
- added D6: 1N914, MyModules:SOD323-C1A2, B.Cu at (232.0, 83.0)
- added D6: 1N914, MyModules:SOD323-C1A2, B.Cu at (167.0, 83.0)
- added D6: 1N914, MyModules:SOD323-C1A2, B.Cu at (102.0, 83.0)
- added D7: 1N914, MyModules:SOD323-C1A2, B.Cu at (262.2, 29.2)
- added D7: 1N914, MyModules:SOD323-C1A2, B.Cu at (197.2, 29.2)
- added D7: 1N914, MyModules:SOD323-C1A2, B.Cu at (132.2, 29.2)
- added D8: S1BB, MyModules:SMB-1C2A, B.Cu at (267.5, 20.2)
- added D8: S1BB, MyModules:SMB-1C2A, B.Cu at (202.5, 20.2)
- added D8: S1BB, MyModules:SMB-1C2A, B.Cu at (137.5, 20.2)
- added D9: S1BB, MyModules:SMB-1C2A, B.Cu at (267.5, 46.8)
- added D9: S1BB, MyModules:SMB-1C2A, B.Cu at (202.5, 46.8)
- added D9: S1BB, MyModules:SMB-1C2A, B.Cu at (137.5, 46.8)
- added J1: PJ301B, MyModules:PJ-301B-JACK-SLOTS, F.Cu at (214.0, 106.5)
- added J1: PJ301B, MyModules:PJ-301B-JACK-SLOTS, F.Cu at (149.0, 106.5)
- added J1: PJ301B, MyModules:PJ-301B-JACK-SLOTS, F.Cu at (84.0, 106.5)
- added J2: PJ301B, MyModules:PJ-301B-JACK-SLOTS, F.Cu at (214.0, 92.5)
- added J2: PJ301B, MyModules:PJ-301B-JACK-SLOTS, F.Cu at (149.0, 92.5)
- added J2: PJ301B, MyModules:PJ-301B-JACK-SLOTS, F.Cu at (84.0, 92.5)
- added J3: PJ301B, MyModules:PJ-301B-JACK-SLOTS, F.Cu at (265.0, 92.5)
- added J3: PJ301B, MyModules:PJ-301B-JACK-SLOTS, F.Cu at (200.0, 92.5)
- added J3: PJ301B, MyModules:PJ-301B-JACK-SLOTS, F.Cu at (135.0, 92.5)
- added J4: PJ301B, MyModules:PJ-301B-JACK-SLOTS, F.Cu at (251.0, 106.5)
- added J4: PJ301B, MyModules:PJ-301B-JACK-SLOTS, F.Cu at (186.0, 106.5)
- added J4: PJ301B, MyModules:PJ-301B-JACK-SLOTS, F.Cu at (121.0, 106.5)
- added J5: PJ301B, MyModules:PJ-301B-JACK-SLOTS, F.Cu at (228.0, 106.5)
- added J5: PJ301B, MyModules:PJ-301B-JACK-SLOTS, F.Cu at (163.0, 106.5)
- added J5: PJ301B, MyModules:PJ-301B-JACK-SLOTS, F.Cu at (98.0, 106.5)
- added J6: PJ301B, MyModules:PJ-301B-JACK-SLOTS, F.Cu at (265.0, 106.5)
- added J6: PJ301B, MyModules:PJ-301B-JACK-SLOTS, F.Cu at (200.0, 106.5)
- added J6: PJ301B, MyModules:PJ-301B-JACK-SLOTS, F.Cu at (135.0, 106.5)
- added P1: CONN_02X05, Pin_Headers:Pin_Header_Straight_2x05, B.Cu at (266.2, 36.5)
- added P1: CONN_02X05, Pin_Headers:Pin_Header_Straight_2x05, B.Cu at (201.2, 36.5)
- added P1: CONN_02X05, Pin_Headers:Pin_Header_Straight_2x05, B.Cu at (136.2, 36.5)
- added Q1: BCM857BS, SMD TRAN:sot323-6, B.Cu at (216.8, 65.2)
- added Q1: BCM857BS, SMD TRAN:sot323-6, B.Cu at (151.8, 65.2)
- added Q1: BCM857BS, SMD TRAN:sot323-6, B.Cu at (86.8, 65.2)
- added Q2: BCM857BS, SMD TRAN:sot323-6, B.Cu at (232.8, 26.0)
- added Q2: BCM857BS, SMD TRAN:sot323-6, B.Cu at (167.8, 26.0)
- added Q2: BCM857BS, SMD TRAN:sot323-6, B.Cu at (102.8, 26.0)
- added Q3: J112, MyModules:SOT23-JRL, B.Cu at (246.0, 66.0)
- added Q3: J112, MyModules:SOT23-JRL, B.Cu at (181.0, 66.0)
- added Q3: J112, MyModules:SOT23-JRL, B.Cu at (116.0, 66.0)
- added Q4: J112, MyModules:SOT23-JRL, B.Cu at (233.0, 66.0)
- added Q4: J112, MyModules:SOT23-JRL, B.Cu at (168.0, 66.0)
- added Q4: J112, MyModules:SOT23-JRL, B.Cu at (103.0, 66.0)
- added Q5: J112, MyModules:SOT23-JRL, B.Cu at (233.0, 96.0)
- added Q5: J112, MyModules:SOT23-JRL, B.Cu at (168.0, 96.0)
- added Q5: J112, MyModules:SOT23-JRL, B.Cu at (103.0, 96.0)
- added Q6: J112, MyModules:SOT23-JRL, B.Cu at (246.0, 96.0)
- added Q6: J112, MyModules:SOT23-JRL, B.Cu at (181.0, 96.0)
- added Q6: J112, MyModules:SOT23-JRL, B.Cu at (116.0, 96.0)
- added R1: 10K, MyModules:SM0603-R-JRL, B.Cu at (225.0, 31.8)
- added R1: 10K, MyModules:SM0603-R-JRL, B.Cu at (160.0, 31.8)
- added R1: 10K, MyModules:SM0603-R-JRL, B.Cu at (95.0, 31.8)
- added R10: 680K, MyModules:SM0603-R-JRL, B.Cu at (221.0, 17.0)
- added R10: 680K, MyModules:SM0603-R-JRL, B.Cu at (156.0, 17.0)
- added R10: 680K, MyModules:SM0603-R-JRL, B.Cu at (91.0, 17.0)
- added R11: 1M, MyModules:SM0603-R-JRL, B.Cu at (216.8, 48.5)
- added R11: 1M, MyModules:SM0603-R-JRL, B.Cu at (151.8, 48.5)
- added R11: 1M, MyModules:SM0603-R-JRL, B.Cu at (86.8, 48.5)
- added R12: 1K, MyModules:SM0603-R-JRL, B.Cu at (220.0, 46.5)
- added R12: 1K, MyModules:SM0603-R-JRL, B.Cu at (155.0, 46.5)
- added R12: 1K, MyModules:SM0603-R-JRL, B.Cu at (90.0, 46.5)
- added R13: 47K, MyModules:SM0603-R-JRL, B.Cu at (226.5, 21.0)
- added R13: 47K, MyModules:SM0603-R-JRL, B.Cu at (161.5, 21.0)
- added R13: 47K, MyModules:SM0603-R-JRL, B.Cu at (96.5, 21.0)
- added R14: 47K, MyModules:SM0603-R-JRL, B.Cu at (236.0, 45.0)
- added R14: 47K, MyModules:SM0603-R-JRL, B.Cu at (171.0, 45.0)
- added R14: 47K, MyModules:SM0603-R-JRL, B.Cu at (106.0, 45.0)
- added R15: 150K, MyModules:SM0603-R-JRL, B.Cu at (216.8, 46.5)
- added R15: 150K, MyModules:SM0603-R-JRL, B.Cu at (151.8, 46.5)
- added R15: 150K, MyModules:SM0603-R-JRL, B.Cu at (86.8, 46.5)
- added R16: 4.7K, MyModules:SM0603-R-JRL, B.Cu at (226.5, 24.0)
- added R16: 4.7K, MyModules:SM0603-R-JRL, B.Cu at (161.5, 24.0)
- added R16: 4.7K, MyModules:SM0603-R-JRL, B.Cu at (96.5, 24.0)
- added R17: 5.6K, MyModules:SM0603-R-JRL, B.Cu at (227.8, 26.8)
- added R17: 5.6K, MyModules:SM0603-R-JRL, B.Cu at (162.8, 26.8)
- added R17: 5.6K, MyModules:SM0603-R-JRL, B.Cu at (97.8, 26.8)
- added R18: 47K, MyModules:SM0603-R-JRL, B.Cu at (239.5, 47.0)
- added R18: 47K, MyModules:SM0603-R-JRL, B.Cu at (174.5, 47.0)
- added R18: 47K, MyModules:SM0603-R-JRL, B.Cu at (109.5, 47.0)
- added R19: 10K NTC, MyModules:SM0805-HAND, B.Cu at (230.0, 26.0)
- added R19: 10K NTC, MyModules:SM0805-HAND, B.Cu at (165.0, 26.0)
- added R19: 10K NTC, MyModules:SM0805-HAND, B.Cu at (100.0, 26.0)
- added R2: 100K, MyModules:SM0603-R-JRL, B.Cu at (223.0, 49.2)
- added R2: 100K, MyModules:SM0603-R-JRL, B.Cu at (158.0, 49.2)
- added R2: 100K, MyModules:SM0603-R-JRL, B.Cu at (93.0, 49.2)
- added R20: 1.5K, MyModules:SM0603-R-JRL, B.Cu at (221.0, 63.2)
- added R20: 1.5K, MyModules:SM0603-R-JRL, B.Cu at (156.0, 63.2)
- added R20: 1.5K, MyModules:SM0603-R-JRL, B.Cu at (91.0, 63.2)
- added R21: 1.5M, MyModules:SM0603-R-JRL, B.Cu at (216.8, 59.2)
- added R21: 1.5M, MyModules:SM0603-R-JRL, B.Cu at (151.8, 59.2)
- added R21: 1.5M, MyModules:SM0603-R-JRL, B.Cu at (86.8, 59.2)
- added R22: 8.2K, MyModules:SM0603-R-JRL, B.Cu at (243.0, 49.0)
- added R22: 8.2K, MyModules:SM0603-R-JRL, B.Cu at (178.0, 49.0)
- added R22: 8.2K, MyModules:SM0603-R-JRL, B.Cu at (113.0, 49.0)
- added R23: 1.8K, MyModules:SM0603-R-JRL, B.Cu at (229.8, 22.5)
- added R23: 1.8K, MyModules:SM0603-R-JRL, B.Cu at (164.8, 22.5)
- added R23: 1.8K, MyModules:SM0603-R-JRL, B.Cu at (99.8, 22.5)
- added R24: 100K, MyModules:SM0603-R-JRL, B.Cu at (246.5, 39.0)
- added R24: 100K, MyModules:SM0603-R-JRL, B.Cu at (181.5, 39.0)
- added R24: 100K, MyModules:SM0603-R-JRL, B.Cu at (116.5, 39.0)
- added R25: 820, MyModules:SM0603-R-JRL, B.Cu at (229.0, 18.5)
- added R25: 820, MyModules:SM0603-R-JRL, B.Cu at (164.0, 18.5)
- added R25: 820, MyModules:SM0603-R-JRL, B.Cu at (99.0, 18.5)
- added R26: 100K, MyModules:SM0603-R-JRL, B.Cu at (246.5, 43.0)
- added R26: 100K, MyModules:SM0603-R-JRL, B.Cu at (181.5, 43.0)
- added R26: 100K, MyModules:SM0603-R-JRL, B.Cu at (116.5, 43.0)
- added R27: 1.5K, MyModules:SM0603-R-JRL, B.Cu at (236.2, 25.2)
- added R27: 1.5K, MyModules:SM0603-R-JRL, B.Cu at (171.2, 25.2)
- added R27: 1.5K, MyModules:SM0603-R-JRL, B.Cu at (106.2, 25.2)
- added R28: 1.5M, MyModules:SM0603-R-JRL, B.Cu at (232.8, 18.8)
- added R28: 1.5M, MyModules:SM0603-R-JRL, B.Cu at (167.8, 18.8)
- added R28: 1.5M, MyModules:SM0603-R-JRL, B.Cu at (102.8, 18.8)
- added R29: 68K, MyModules:SM0603-R-JRL, B.Cu at (246.5, 55.5)
- added R29: 68K, MyModules:SM0603-R-JRL, B.Cu at (181.5, 55.5)
- added R29: 68K, MyModules:SM0603-R-JRL, B.Cu at (116.5, 55.5)
- added R3: 100K, MyModules:SM0603-R-JRL, B.Cu at (219.8, 28.5)
- added R3: 100K, MyModules:SM0603-R-JRL, B.Cu at (154.8, 28.5)
- added R3: 100K, MyModules:SM0603-R-JRL, B.Cu at (89.8, 28.5)
- added R30: 560, MyModules:SM0603-R-JRL, B.Cu at (246.5, 58.0)
- added R30: 560, MyModules:SM0603-R-JRL, B.Cu at (181.5, 58.0)
- added R30: 560, MyModules:SM0603-R-JRL, B.Cu at (116.5, 58.0)
- added R31: 18K, MyModules:SM0603-R-JRL, B.Cu at (218.5, 68.0)
- added R31: 18K, MyModules:SM0603-R-JRL, B.Cu at (153.5, 68.0)
- added R31: 18K, MyModules:SM0603-R-JRL, B.Cu at (88.5, 68.0)
- added R32: 18K, MyModules:SM0603-R-JRL, B.Cu at (241.5, 54.0)
- added R32: 18K, MyModules:SM0603-R-JRL, B.Cu at (176.5, 54.0)
- added R32: 18K, MyModules:SM0603-R-JRL, B.Cu at (111.5, 54.0)
- added R33: 33K, MyModules:SM0603-R-JRL, B.Cu at (229.5, 56.5)
- added R33: 33K, MyModules:SM0603-R-JRL, B.Cu at (164.5, 56.5)
- added R33: 33K, MyModules:SM0603-R-JRL, B.Cu at (99.5, 56.5)
- added R34: 33K, MyModules:SM0603-R-JRL, B.Cu at (223.5, 71.5)
- added R34: 33K, MyModules:SM0603-R-JRL, B.Cu at (158.5, 71.5)
- added R34: 33K, MyModules:SM0603-R-JRL, B.Cu at (93.5, 71.5)
- added R35: 68K, MyModules:SM0603-R-JRL, B.Cu at (223.5, 73.5)
- added R35: 68K, MyModules:SM0603-R-JRL, B.Cu at (158.5, 73.5)
- added R35: 68K, MyModules:SM0603-R-JRL, B.Cu at (93.5, 73.5)
- added R36: 560, MyModules:SM0603-R-JRL, B.Cu at (223.5, 75.5)
- added R36: 560, MyModules:SM0603-R-JRL, B.Cu at (158.5, 75.5)
- added R36: 560, MyModules:SM0603-R-JRL, B.Cu at (93.5, 75.5)
- added R37: 68K, MyModules:SM0603-R-JRL, B.Cu at (232.5, 56.5)
- added R37: 68K, MyModules:SM0603-R-JRL, B.Cu at (167.5, 56.5)
- added R37: 68K, MyModules:SM0603-R-JRL, B.Cu at (102.5, 56.5)
- added R38: 560, MyModules:SM0603-R-JRL, B.Cu at (232.5, 54.0)
- added R38: 560, MyModules:SM0603-R-JRL, B.Cu at (167.5, 54.0)
- added R38: 560, MyModules:SM0603-R-JRL, B.Cu at (102.5, 54.0)
- added R39: 18K, MyModules:SM0603-R-JRL, B.Cu at (237.5, 54.0)
- added R39: 18K, MyModules:SM0603-R-JRL, B.Cu at (172.5, 54.0)
- added R39: 18K, MyModules:SM0603-R-JRL, B.Cu at (107.5, 54.0)
- added R4: 100K, MyModules:SM0603-R-JRL, B.Cu at (212.8, 56.2)
- added R4: 100K, MyModules:SM0603-R-JRL, B.Cu at (147.8, 56.2)
- added R4: 100K, MyModules:SM0603-R-JRL, B.Cu at (82.8, 56.2)
- added R40: 33K, MyModules:SM0603-R-JRL, B.Cu at (232.5, 70.5)
- added R40: 33K, MyModules:SM0603-R-JRL, B.Cu at (167.5, 70.5)
- added R40: 33K, MyModules:SM0603-R-JRL, B.Cu at (102.5, 70.5)
- added R41: 3.3K, MyModules:SM0603-R-JRL, B.Cu at (244.0, 16.0)
- added R41: 3.3K, MyModules:SM0603-R-JRL, B.Cu at (179.0, 16.0)
- added R41: 3.3K, MyModules:SM0603-R-JRL, B.Cu at (114.0, 16.0)
- added R42: 56K, MyModules:SM0603-R-JRL, B.Cu at (232.5, 72.5)
- added R42: 56K, MyModules:SM0603-R-JRL, B.Cu at (167.5, 72.5)
- added R42: 56K, MyModules:SM0603-R-JRL, B.Cu at (102.5, 72.5)
- added R43: 56K, MyModules:SM0603-R-JRL, B.Cu at (250.0, 55.5)
- added R43: 56K, MyModules:SM0603-R-JRL, B.Cu at (185.0, 55.5)
- added R43: 56K, MyModules:SM0603-R-JRL, B.Cu at (120.0, 55.5)
- added R44: 100K, MyModules:SM0603-R-JRL, B.Cu at (232.5, 75.5)
- added R44: 100K, MyModules:SM0603-R-JRL, B.Cu at (167.5, 75.5)
- added R44: 100K, MyModules:SM0603-R-JRL, B.Cu at (102.5, 75.5)
- added R45: 100K, MyModules:SM0603-R-JRL, B.Cu at (228.0, 85.5)
- added R45: 100K, MyModules:SM0603-R-JRL, B.Cu at (163.0, 85.5)
- added R45: 100K, MyModules:SM0603-R-JRL, B.Cu at (98.0, 85.5)
- added R46: 33K, MyModules:SM0603-R-JRL, B.Cu at (232.5, 77.5)
- added R46: 33K, MyModules:SM0603-R-JRL, B.Cu at (167.5, 77.5)
- added R46: 33K, MyModules:SM0603-R-JRL, B.Cu at (102.5, 77.5)
- added R47: 100K, MyModules:SM0603-R-JRL, B.Cu at (246.5, 79.5)
- added R47: 100K, MyModules:SM0603-R-JRL, B.Cu at (181.5, 79.5)
- added R47: 100K, MyModules:SM0603-R-JRL, B.Cu at (116.5, 79.5)
- added R48: 100K, MyModules:SM0603-R-JRL, B.Cu at (232.5, 85.5)
- added R48: 100K, MyModules:SM0603-R-JRL, B.Cu at (167.5, 85.5)
- added R48: 100K, MyModules:SM0603-R-JRL, B.Cu at (102.5, 85.5)
- added R49: 10K, MyModules:SM0603-R-JRL, B.Cu at (228.0, 81.5)
- added R49: 10K, MyModules:SM0603-R-JRL, B.Cu at (163.0, 81.5)
- added R49: 10K, MyModules:SM0603-R-JRL, B.Cu at (98.0, 81.5)
- added R5: 200K, MyModules:SM0603-R-JRL, B.Cu at (218.0, 30.5)
- added R5: 200K, MyModules:SM0603-R-JRL, B.Cu at (153.0, 30.5)
- added R5: 200K, MyModules:SM0603-R-JRL, B.Cu at (88.0, 30.5)
- added R50: 47K, MyModules:SM0603-R-JRL, B.Cu at (228.5, 95.5)
- added R50: 47K, MyModules:SM0603-R-JRL, B.Cu at (163.5, 95.5)
- added R50: 47K, MyModules:SM0603-R-JRL, B.Cu at (98.5, 95.5)
- added R51: 100K, MyModules:SM0603-R-JRL, B.Cu at (246.5, 82.0)
- added R51: 100K, MyModules:SM0603-R-JRL, B.Cu at (181.5, 82.0)
- added R51: 100K, MyModules:SM0603-R-JRL, B.Cu at (116.5, 82.0)
- added R52: 68K, MyModules:SM0603-R-JRL, B.Cu at (232.5, 87.5)
- added R52: 68K, MyModules:SM0603-R-JRL, B.Cu at (167.5, 87.5)
- added R52: 68K, MyModules:SM0603-R-JRL, B.Cu at (102.5, 87.5)
- added R53: 560, MyModules:SM0603-R-JRL, B.Cu at (228.0, 87.5)
- added R53: 560, MyModules:SM0603-R-JRL, B.Cu at (163.0, 87.5)
- added R53: 560, MyModules:SM0603-R-JRL, B.Cu at (98.0, 87.5)
- added R54: 1K, MyModules:SM0603-R-JRL, B.Cu at (261.5, 99.0)
- added R54: 1K, MyModules:SM0603-R-JRL, B.Cu at (196.5, 99.0)
- added R54: 1K, MyModules:SM0603-R-JRL, B.Cu at (131.5, 99.0)
- added R55: 18K, MyModules:SM0603-R-JRL, B.Cu at (215.0, 68.0)
- added R55: 18K, MyModules:SM0603-R-JRL, B.Cu at (150.0, 68.0)
- added R55: 18K, MyModules:SM0603-R-JRL, B.Cu at (85.0, 68.0)
- added R56: 18K, MyModules:SM0603-R-JRL, B.Cu at (237.5, 85.2)
- added R56: 18K, MyModules:SM0603-R-JRL, B.Cu at (172.5, 85.2)
- added R56: 18K, MyModules:SM0603-R-JRL, B.Cu at (107.5, 85.2)
- added R57: 33K, MyModules:SM0603-R-JRL, B.Cu at (228.5, 97.5)
- added R57: 33K, MyModules:SM0603-R-JRL, B.Cu at (163.5, 97.5)
- added R57: 33K, MyModules:SM0603-R-JRL, B.Cu at (98.5, 97.5)
- added R58: 33K, MyModules:SM0603-R-JRL, B.Cu at (256.2, 32.5)
- added R58: 33K, MyModules:SM0603-R-JRL, B.Cu at (191.2, 32.5)
- added R58: 33K, MyModules:SM0603-R-JRL, B.Cu at (126.2, 32.5)
- added R59: 330, MyModules:SM0603-R-JRL, B.Cu at (260.2, 32.8)
- added R59: 330, MyModules:SM0603-R-JRL, B.Cu at (195.2, 32.8)
- added R59: 330, MyModules:SM0603-R-JRL, B.Cu at (130.2, 32.8)
- added R6: 200K, MyModules:SM0603-R-JRL, B.Cu at (218.0, 26.5)
- added R6: 200K, MyModules:SM0603-R-JRL, B.Cu at (153.0, 26.5)
- added R6: 200K, MyModules:SM0603-R-JRL, B.Cu at (88.0, 26.5)
- added R60: 68K, MyModules:SM0603-R-JRL, B.Cu at (210.5, 73.5)
- added R60: 68K, MyModules:SM0603-R-JRL, B.Cu at (145.5, 73.5)
- added R60: 68K, MyModules:SM0603-R-JRL, B.Cu at (80.5, 73.5)
- added R61: 100K, MyModules:SM0603-R-JRL, B.Cu at (260.2, 29.2)
- added R61: 100K, MyModules:SM0603-R-JRL, B.Cu at (195.2, 29.2)
- added R61: 100K, MyModules:SM0603-R-JRL, B.Cu at (130.2, 29.2)
- added R62: 560, MyModules:SM0603-R-JRL, B.Cu at (210.5, 71.5)
- added R62: 560, MyModules:SM0603-R-JRL, B.Cu at (145.5, 71.5)
- added R62: 560, MyModules:SM0603-R-JRL, B.Cu at (80.5, 71.5)
- added R63: 68K, MyModules:SM0603-R-JRL, B.Cu at (237.0, 98.0)
- added R63: 68K, MyModules:SM0603-R-JRL, B.Cu at (172.0, 98.0)
- added R63: 68K, MyModules:SM0603-R-JRL, B.Cu at (107.0, 98.0)
- added R64: 330, MyModules:SM0603-R-JRL, B.Cu at (256.2, 29.5)
- added R64: 330, MyModules:SM0603-R-JRL, B.Cu at (191.2, 29.5)
- added R64: 330, MyModules:SM0603-R-JRL, B.Cu at (126.2, 29.5)
- added R65: 560, MyModules:SM0603-R-JRL, B.Cu at (237.0, 100.0)
- added R65: 560, MyModules:SM0603-R-JRL, B.Cu at (172.0, 100.0)
- added R65: 560, MyModules:SM0603-R-JRL, B.Cu at (107.0, 100.0)
- added R66: 10, MyModules:SM0805-HAND, B.Cu at (267.5, 23.5)
- added R66: 10, MyModules:SM0805-HAND, B.Cu at (202.5, 23.5)
- added R66: 10, MyModules:SM0805-HAND, B.Cu at (137.5, 23.5)
- added R67: 10, MyModules:SM0805-HAND, B.Cu at (267.8, 43.2)
- added R67: 10, MyModules:SM0805-HAND, B.Cu at (202.8, 43.2)
- added R67: 10, MyModules:SM0805-HAND, B.Cu at (137.8, 43.2)
- added R68: 18K, MyModules:SM0603-R-JRL, B.Cu at (241.5, 85.2)
- added R68: 18K, MyModules:SM0603-R-JRL, B.Cu at (176.5, 85.2)
- added R68: 18K, MyModules:SM0603-R-JRL, B.Cu at (111.5, 85.2)
- added R69: 33K, MyModules:SM0603-R-JRL, B.Cu at (242.0, 98.0)
- added R69: 33K, MyModules:SM0603-R-JRL, B.Cu at (177.0, 98.0)
- added R69: 33K, MyModules:SM0603-R-JRL, B.Cu at (112.0, 98.0)
- added R7: 100K, MyModules:SM0603-R-JRL, B.Cu at (235.0, 41.2)
- added R7: 100K, MyModules:SM0603-R-JRL, B.Cu at (170.0, 41.2)
- added R7: 100K, MyModules:SM0603-R-JRL, B.Cu at (105.0, 41.2)
- added R70: 10K, MyModules:SM0603-R-JRL, B.Cu at (246.5, 75.5)
- added R70: 10K, MyModules:SM0603-R-JRL, B.Cu at (181.5, 75.5)
- added R70: 10K, MyModules:SM0603-R-JRL, B.Cu at (116.5, 75.5)
- added R71: 10K, MyModules:SM0603-R-JRL, B.Cu at (246.5, 71.5)
- added R71: 10K, MyModules:SM0603-R-JRL, B.Cu at (181.5, 71.5)
- added R71: 10K, MyModules:SM0603-R-JRL, B.Cu at (116.5, 71.5)
- added R72: 10K, MyModules:SM0603-R-JRL, B.Cu at (246.5, 73.5)
- added R72: 10K, MyModules:SM0603-R-JRL, B.Cu at (181.5, 73.5)
- added R72: 10K, MyModules:SM0603-R-JRL, B.Cu at (116.5, 73.5)
- added R73: 100K, MyModules:SM0603-R-JRL, B.Cu at (223.0, 52.5)
- added R73: 100K, MyModules:SM0603-R-JRL, B.Cu at (158.0, 52.5)
- added R73: 100K, MyModules:SM0603-R-JRL, B.Cu at (93.0, 52.5)
- added R74: 100K, MyModules:SM0603-R-JRL, B.Cu at (212.8, 53.2)
- added R74: 100K, MyModules:SM0603-R-JRL, B.Cu at (147.8, 53.2)
- added R74: 100K, MyModules:SM0603-R-JRL, B.Cu at (82.8, 53.2)
- added R75: 100K, MyModules:SM0603-R-JRL, B.Cu at (219.0, 50.5)
- added R75: 100K, MyModules:SM0603-R-JRL, B.Cu at (154.0, 50.5)
- added R75: 100K, MyModules:SM0603-R-JRL, B.Cu at (89.0, 50.5)
- added R76: 100K, MyModules:SM0603-R-JRL, B.Cu at (212.8, 21.8)
- added R76: 100K, MyModules:SM0603-R-JRL, B.Cu at (147.8, 21.8)
- added R76: 100K, MyModules:SM0603-R-JRL, B.Cu at (82.8, 21.8)
- added R77: 100K, MyModules:SM0603-R-JRL, B.Cu at (216.0, 21.8)
- added R77: 100K, MyModules:SM0603-R-JRL, B.Cu at (151.0, 21.8)
- added R77: 100K, MyModules:SM0603-R-JRL, B.Cu at (86.0, 21.8)
- added R78: 100K, MyModules:SM0603-R-JRL, B.Cu at (221.0, 19.0)
- added R78: 100K, MyModules:SM0603-R-JRL, B.Cu at (156.0, 19.0)
- added R78: 100K, MyModules:SM0603-R-JRL, B.Cu at (91.0, 19.0)
- added R8: 100K, MyModules:SM0603-R-JRL, B.Cu at (236.0, 49.0)
- added R8: 100K, MyModules:SM0603-R-JRL, B.Cu at (171.0, 49.0)
- added R8: 100K, MyModules:SM0603-R-JRL, B.Cu at (106.0, 49.0)
- added R9: 110K, MyModules:SM0603-R-JRL, B.Cu at (220.0, 48.5)
- added R9: 110K, MyModules:SM0603-R-JRL, B.Cu at (155.0, 48.5)
- added R9: 110K, MyModules:SM0603-R-JRL, B.Cu at (90.0, 48.5)
- added REF**: fiducial-1mm, MyModules:fiducial-1mm, B.Cu at (269.5, 109.5)
- added REF**: fiducial-2mm, MyModules:fiducial-2mm, B.Cu at (277.0, 7.00)
- added REF**: fiducial-2mm, MyModules:fiducial-2mm, B.Cu at (277.0, 117.0)
- added REF**: fiducial-2mm, MyModules:fiducial-2mm, B.Cu at (7.00, 117.0)
- added REF**: fiducial-1mm, MyModules:fiducial-1mm, B.Cu at (210.0, 15.0)
- added REF**: fiducial-1mm, MyModules:fiducial-1mm, B.Cu at (204.5, 109.5)
- added REF**: fiducial-1mm, MyModules:fiducial-1mm, B.Cu at (145.0, 15.0)
- added REF**: fiducial-1mm, MyModules:fiducial-1mm, B.Cu at (80.0, 15.0)
- added REF**: fiducial-1mm, MyModules:fiducial-1mm, B.Cu at (139.5, 109.5)
- added REF**: fiducial-2mm, MyModules:fiducial-2mm, B.Cu at (7.00, 7.00)
- added SW1: KS-01Q, synth:KS-01Q-02-JRL, F.Cu at (192.0, 20.5)
- added SW1: KS-01Q, synth:KS-01Q-02-JRL, F.Cu at (257.0, 20.5)
- added SW1: KS-01Q, synth:KS-01Q-02-JRL, F.Cu at (127.0, 20.5)
- added TP1: TEST_POINT, MyModules:TEST POINT, B.Cu at (219.2, 43.5)
- added TP1: TEST_POINT, MyModules:TEST POINT, B.Cu at (154.2, 43.5)
- added TP1: TEST_POINT, MyModules:TEST POINT, B.Cu at (89.2, 43.5)
- added TP2: TEST_POINT, MyModules:TEST POINT, B.Cu at (226.5, 16.2)
- added TP2: TEST_POINT, MyModules:TEST POINT, B.Cu at (161.5, 16.2)
- added TP2: TEST_POINT, MyModules:TEST POINT, B.Cu at (96.5, 16.2)
- added U1: TL072-, MyModules:TSSOP8-JRL, B.Cu at (221.2, 21.8)
- added U1: TL072-, MyModules:TSSOP8-JRL, B.Cu at (156.2, 21.8)
- added U1: TL072-, MyModules:TSSOP8-JRL, B.Cu at (91.2, 21.8)
- added U10: CD4027, Housings_SSOP:TSSOP-16_4.4x5mm_Pitch0.65mm, B.Cu at (259.0, 44.0)
- added U10: CD4027, Housings_SSOP:TSSOP-16_4.4x5mm_Pitch0.65mm, B.Cu at (194.0, 44.0)
- added U10: CD4027, Housings_SSOP:TSSOP-16_4.4x5mm_Pitch0.65mm, B.Cu at (129.0, 44.0)
- added U11: CD40106, Housings_SSOP:TSSOP-14_4.4x5mm_Pitch0.65mm, B.Cu at (259.0, 37.5)
- added U11: CD40106, Housings_SSOP:TSSOP-14_4.4x5mm_Pitch0.65mm, B.Cu at (194.0, 37.5)
- added U11: CD40106, Housings_SSOP:TSSOP-14_4.4x5mm_Pitch0.65mm, B.Cu at (129.0, 37.5)
- added U12: TS321, TO_SOT_Packages_SMD:SOT-23-5, B.Cu at (216.8, 62.2)
- added U12: TS321, TO_SOT_Packages_SMD:SOT-23-5, B.Cu at (151.8, 62.2)
- added U12: TS321, TO_SOT_Packages_SMD:SOT-23-5, B.Cu at (86.8, 62.2)
- added U13: TS321, TO_SOT_Packages_SMD:SOT-23-5, B.Cu at (232.8, 23.0)
- added U13: TS321, TO_SOT_Packages_SMD:SOT-23-5, B.Cu at (167.8, 23.0)
- added U13: TS321, TO_SOT_Packages_SMD:SOT-23-5, B.Cu at (102.8, 23.0)
- added U2: TL072-, MyModules:TSSOP8-JRL, B.Cu at (218.2, 53.0)
- added U2: TL072-, MyModules:TSSOP8-JRL, B.Cu at (153.2, 53.0)
- added U2: TL072-, MyModules:TSSOP8-JRL, B.Cu at (88.2, 53.0)
- added U3: TL072-, MyModules:TSSOP8-JRL, B.Cu at (239.6, 42.0)
- added U3: TL072-, MyModules:TSSOP8-JRL, B.Cu at (174.6, 42.0)
- added U3: TL072-, MyModules:TSSOP8-JRL, B.Cu at (109.6, 42.0)
- added U4: TL072-, MyModules:TSSOP8-JRL, B.Cu at (239.3, 81.5)
- added U4: TL072-, MyModules:TSSOP8-JRL, B.Cu at (174.3, 81.5)
- added U4: TL072-, MyModules:TSSOP8-JRL, B.Cu at (109.3, 81.5)
- added U5: LM13700, MyModules:SO16-JRL, B.Cu at (239.5, 60.5)
- added U5: LM13700, MyModules:SO16-JRL, B.Cu at (174.5, 60.5)
- added U5: LM13700, MyModules:SO16-JRL, B.Cu at (109.5, 60.5)
- added U6: LM13700, MyModules:SO16-JRL, B.Cu at (217.0, 74.5)
- added U6: LM13700, MyModules:SO16-JRL, B.Cu at (152.0, 74.5)
- added U6: LM13700, MyModules:SO16-JRL, B.Cu at (87.0, 74.5)
- added U7: LM13700, MyModules:SO16-JRL, B.Cu at (239.5, 91.5)
- added U7: LM13700, MyModules:SO16-JRL, B.Cu at (174.5, 91.5)
- added U7: LM13700, MyModules:SO16-JRL, B.Cu at (109.5, 91.5)
- added U8: DG409, MyModules:SO16-JRL, B.Cu at (239.5, 74.5)
- added U8: DG409, MyModules:SO16-JRL, B.Cu at (174.5, 74.5)
- added U8: DG409, MyModules:SO16-JRL, B.Cu at (109.5, 74.5)
- added U9: CD4052, Housings_SSOP:TSSOP-16_4.4x5mm_Pitch0.65mm, B.Cu at (247.5, 20.5)
- added U9: CD4052, Housings_SSOP:TSSOP-16_4.4x5mm_Pitch0.65mm, B.Cu at (182.5, 20.5)
- added U9: CD4052, Housings_SSOP:TSSOP-16_4.4x5mm_Pitch0.65mm, B.Cu at (117.5, 20.5)
- added VR1: 50K, MyModules:RV16A-41-JRL, F.Cu at (222.0, 20.5)
- added VR1: 50K, MyModules:RV16A-41-JRL, F.Cu at (157.0, 20.5)
- added VR1: 50K, MyModules:RV16A-41-JRL, F.Cu at (92.0, 20.5)
- added VR2: 50K, MyModules:RV16A-41-JRL, F.Cu at (157.0, 46.5)
- added VR2: 50K, MyModules:RV16A-41-JRL, F.Cu at (222.0, 46.5)
- added VR2: 50K, MyModules:RV16A-41-JRL, F.Cu at (92.0, 46.5)
- added VR3: 50K, MyModules:RV16A-41-JRL, F.Cu at (222.0, 72.5)
- added VR3: 50K, MyModules:RV16A-41-JRL, F.Cu at (157.0, 72.5)
- added VR3: 50K, MyModules:RV16A-41-JRL, F.Cu at (92.0, 72.5)
- added VR4: 50K, MyModules:RV16A-41-JRL, F.Cu at (257.0, 72.5)
- added VR4: 50K, MyModules:RV16A-41-JRL, F.Cu at (192.0, 72.5)
- added VR4: 50K, MyModules:RV16A-41-JRL, F.Cu at (127.0, 72.5)
- added VR5: 100K, MyModules:TC33X-2, B.Cu at (212.8, 28.0)
- added VR5: 100K, MyModules:TC33X-2, B.Cu at (147.8, 28.0)
- added VR5: 100K, MyModules:TC33X-2, B.Cu at (82.8, 28.0)
- added VR6: 50K, MyModules:RV16A-41-JRL, F.Cu at (192.0, 46.5)
- added VR6: 50K, MyModules:RV16A-41-JRL, F.Cu at (257.0, 46.5)
- added VR6: 50K, MyModules:RV16A-41-JRL, F.Cu at (127.0, 46.5)
- added VR7: 100K, MyModules:TC33X-2, B.Cu at (212.8, 46.0)
- added VR7: 100K, MyModules:TC33X-2, B.Cu at (147.8, 46.0)
- added VR7: 100K, MyModules:TC33X-2, B.Cu at (82.8, 46.0)
Routing:
- net +12V: track 493.8 -> 1975.2 mm, vias 20 -> 80
- net -12V: track 337.3 -> 1349.4 mm, vias 18 -> 72
- net FREQ_CTRL: track 105.1 -> 420.5 mm
- net Net-(U10-Pad1): track 94.4 -> 377.6 mm, vias 4 -> 16
- net Net-(C3-Pad2): track 83.9 -> 335.7 mm
- net Net-(U10-Pad15): track 81.0 -> 323.9 mm
- net Net-(J4-Pad3): track 74.2 -> 296.8 mm
- net Net-(R3-Pad2): track 72.5 -> 289.9 mm, vias 1 -> 4
- net Net-(J2-Pad3): track 70.0 -> 279.9 mm
- net Net-(C8-Pad1): track 65.0 -> 260.1 mm, vias 3 -> 12
- net Net-(J5-Pad3): track 62.4 -> 249.4 mm, vias 1 -> 4
- net Net-(C3-Pad1): track 62.3 -> 249.0 mm, vias 3 -> 12
- net Net-(J1-Pad3): track 47.0 -> 187.9 mm, vias 1 -> 4
- net GND: track 45.8 -> 183.1 mm, vias 20 -> 80
- net Net-(Q5-Pad1): track 44.3 -> 177.1 mm
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Other:
- board outline removed

Commit message: generated gerbers for review by assembler
Parts:
- added REF***: OSHW-Symbol_6.7x6mm_SilkScreen, Symbols:OSHW-Symbol_6.7x6mm_SilkScreen, B.Cu at (44.2, 107.0)
- added REF***: OSHW-Symbol_6.7x6mm_SilkScreen, Symbols:OSHW-Symbol_6.7x6mm_SilkScreen, B.Cu at (109.2, 107.0)
- added REF***: OSHW-Symbol_6.7x6mm_SilkScreen, Symbols:OSHW-Symbol_6.7x6mm_SilkScreen, B.Cu at (174.2, 107.0)
- added REF***: OSHW-Symbol_6.7x6mm_SilkScreen, Symbols:OSHW-Symbol_6.7x6mm_SilkScreen, B.Cu at (239.2, 107.0)
Other:
- board outline added: 280 x 120 mm
